File: ki_cad_project/farseer/3v3_cell.kicad_sch (KiCad schematic)
At the start: 18 parts, among them U3 TPS54560-Q1

Commit message: finished rev1
Parts:
- U3: DigikeyPN (none) -> 296-38302-1-ND; DigikeyURL (none) -> https://www.digikey.com/en/products/detail/texas-instrument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
Changed lines of the file:
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@@
 			)
 		)
-		(property "Description" "Buck converter, 4.5-60V in, 5A, non-synchronous, adjustable frequency, AEC-Q100, 3V3_CELL rail (U2), HSOIC-8 PowerPAD (DDA)"
+		(property "Description" "Buck converter, 4.5-60V in, 5A, non-synchronous, adjustable frequency, AEC-Q100, 3V3_CELL rail (U3), HSOIC-8 PowerPAD (DDA)"
 			(at 134.62 104.14 0)
 			(hide yes)
@@
 			(hide yes)
 			(show_name no)
+			(do_not_autoplace no)
+			(effects
+				(font
+					(size 1.27 1.27)
+				)
+			)
+		)
+		(property "DigikeyPN" "296-38302-1-ND"
+			(at 134.62 86.36 0)
+			(hide yes)
+			(show_name no)
+			(do_not_autoplace no)
+			(effects
+				(font
+					(size 1.27 1.27)
+				)
+			)
+		)
+		(property "DigikeyURL" "https://www.digikey.com/en/products/detail/texas-instruments/TPS54560QDDARQ1/4476064?s=N4IgTCBcDa4JwDYC0BmAHCgDGJBGJAcgCIgC6AvkA"
+			(at 134.62 86.36 0)
+			(hide yes)
+			(show_name no)
