File: ki_cad_project/farseer/3v3_sys.kicad_sch (KiCad schematic)
At the start: 10 parts, among them U2 LMR16006X

Commit message: finished rev1
Parts:
- added R51: 100k, Resistor_SMD:R_0603_1608Metric, symbol Device:R_US
Connections:
- net +12VF: now also R51.1; no longer U2.4 (SHDN)
- new net: R51.2, U2.4 (SHDN)
Changed lines of the file:
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@@
 	)
 	(junction
-		(at 133.35 95.25)
+		(at 129.54 95.25)
 		(diameter 0)
 		(color 0 0 0 0)
@@
 	(wire
 		(pts
-			(xy 133.35 95.25) (xy 133.35 100.33)
-		)
-		(stroke
-			(width 0)
-			(type default)
-		)
-	)
-	(wire
-		(pts
 			(xy 209.55 106.68) (xy 209.55 107.95)
 		)
@@
 	(wire
 		(pts
+			(xy 132.08 100.33) (xy 133.35 100.33)
+		)
+		(stroke
+			(width 0)
+			(type default)
+		)
+	)
+	(wire
+		(pts
 			(xy 165.1 105.41) (xy 165.1 106.68)
 		)
@@
 	(wire
 		(pts
+			(xy 129.54 95.25) (xy 129.54 107.95)
+		)
+		(stroke
+			(width 0)
+			(type default)
+		)
+	)
+	(wire
+		(pts
 			(xy 180.34 97.79) (xy 184.15 97.79)
 		)
@@
 	(wire
 		(pts
+			(xy 129.54 107.95) (xy 132.08 107.95)
+		)
+		(stroke
+			(width 0)
+			(type default)
+		)
+	)
+	(wire
+		(pts
 			(xy 204.47 106.68) (xy 209.55 106.68)
 		)
@@
 	(wire
 		(pts
-			(xy 125.73 95.25) (xy 133.35 95.25)
+			(xy 125.73 95.25) (xy 129.54 95.25)
+		)
+		(stroke
+			(width 0)
+			(type default)
+		)
+	)
+	(wire
+		(pts
+			(xy 129.54 95.25) (xy 133.35 95.25)
 		)
 		(stroke
@@
 			(width 0)
 			(type default)
+		)
+	)
+	(symbol
+		(lib_id "Device:R_US")
+		(at 132.08 104.14 180)
+		(unit 1)
+		(body_style 1)
+		(exclude_from_sim no)
+		(in_bom yes)
+		(on_board yes)
+		(in_pos_files yes)
+		(dnp no)
+		(property "Reference" "R51"
+			(at 135.636 103.124 0)
+			(show_name no)
+			(do_not_autoplace no)
+			(effects
+				(font
+					(size 1.27 1.27)
+				)
+			)
+		)
+		(property "Value" "100k"
+			(at 135.636 105.156 0)
+			(show_name no)
+			(do_not_autoplace no)
+			(effects
+				(font
+					(size 1.27 1.27)
+				)
+			)
+		)
+		(property "Footprint" "Resistor_SMD:R_0603_1608Metric"
+			(at 131.064 103.886 90)
+			(hide yes)
+			(show_name no)
+			(do_not_autoplace no)
+			(effects
+				(font
+					(size 1.27 1.27)
+				)
+			)
+		)
+		(property "Datasheet" ""
+			(at 132.08 104.14 0)
+			(hide yes)
+			(show_name no)
+			(do_not_autoplace no)
+			(effects
+				(font
+					(size 1.27 1.27)
+				)
+			)
+		)
+		(property "Description" "Resistor, US symbol"
+			(at 132.08 104.14 0)
+			(hide yes)
+			(show_name no)
+			(do_not_autoplace no)
+			(effects
+				(font
+					(size 1.27 1.27)
+				)
+			)
+		)
+		(property "MPN" "AC0603FR-07100KL"
+			(at 132.08 104.14 0)
+			(hide yes)
+			(show_name no)
+			(do_not_autoplace no)
+			(effects
+				(font
+					(size 1.27 1.27)
+				)
+			)
+		)
+		(property "Manufacturer" "Yageo"
+			(at 132.08 104.14 0)
+			(hide yes)
+			(show_name no)
+			(do_not_autoplace no)
+			(effects
+				(font
+					(size 1.27 1.27)
+				)
+			)
+		)
+		(property "Design Notes" "Series resistor between +12VF and U2 SHDN. LMR16006 datasheet sec 8.3.4: when shutdown is not used the pin 'may be tied to VIN via 100 kOhm resistor', and 100 kOhm or larger is recommended whenever a voltage above logic level is applied 'to protect the device'. SHDN abs max is 65 V and the SM8S26A clamp on +12VF is ~42 V, so this is datasheet compliance rather than transient survival. SHDN rising threshold 1.25 V typ; the internal pull-up current (about 1-4 uA) drops well under 0.5 V across 100k, so U2 is enabled at every valid input voltage."
+			(at 132.08 104.14 0)
+			(hide yes)
+			(show_name no)
+			(do_not_autoplace no)
+			(effects
+				(font
+					(size 1.27 1.27)
+				)
+			)
+		)
+		(pin "1"
+		)
+		(pin "2"
+		)
+		(instances
+			(project "farseer"
+				(path "/b50562dd-c7d3-426b-8c59-03f29968ae16/86904090-babb-411a-8c68-882bbb5c2231"
+					(reference "R51")
+					(unit 1)
+				)
+			)
 		)
 	)
@@
 		(dnp no)
 		(property "Reference" "C38"
-			(at 128.27 97.79 0)
+			(at 121.412 101.6 0)
 			(show_name no)
 			(do_not_autoplace no)
@@
 		)
 		(property "Value" "0u1"
-			(at 128.27 99.568 0)
+			(at 121.412 103.378 0)
 			(show_name no)
 			(do_not_autoplace no)
@@
 		(dnp no)
 		(property "Reference" "C37"
-			(at 118.11 97.79 0)
+			(at 110.49 101.854 0)
 			(show_name no)
 			(do_not_autoplace no)
@@
 		)
 		(property "Value" "4u7"
-			(at 118.11 99.568 0)
-			(show_name no)
-			(do_not_autoplace no)
+			(at 110.49 103.632 0)
+			(show_name no)
+			(do_not_autoplace no)
