File: ki_cad_project/farseer/cellular.kicad_sch (KiCad schematic)
At the start: 20 parts, among them J5 BG95-M3_MiniPCIe, J6 SIM8060-6-1-14-00, U9 TPD4E02B04DQA

Commit message: finished rev1
Parts:
- U9: MPN (none) -> TPD4E02B04DQAR; Manufacturer (none) -> Texas Instruments
Changed lines of the file:
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@@
 			)
 		)
-		(property "MPN" ""
+		(property "MPN" "TPD4E02B04DQAR"
 			(at 240.03 92.71 0)
 			(hide yes)
@@
 			)
 		)
-		(property "Manufacturer" ""
+		(property "Manufacturer" "Texas Instruments"
 			(at 240.03 92.71 0)
 			(hide yes)
