File: ki_cad_project/farseer/farseer.kicad_pcb (KiCad board)
At the start: 4 copper layers, 100 x 130 mm, 112 parts, among them J1 Conn_PIC_ICSP_ICD, J2 Conn_01x02, J3 SMA_RA_TH_50R, J4 USB_C_Receptacle_USB2.0_16P, J5 BG95-M3_MiniPCIe, J6 SIM8060-6-1-14-00, Q1 DMP6023LFGQ, U1 PIC18F57Q84, U2 LMR16006X, U3 TPS54560-Q1, U4 NEO-M9N, U6 USBLC6-2SC6, U7 CP2102N-Axx-xQFN24, U9 TPD4E02B04DQA

Commit message: finished rev1
Parts:
- added R51: 100k, Resistor_SMD:R_0603_1608Metric, F.Cu at (71.7, 49.2)
- J1: footprint Connector_PinHeader_2.54mm:PinHeader_1x06_P2.54mm_Horizontal -> Connector_PinHeader_2.54mm:PinHeader_1x06_P2.54mm_Vertical
- moved C45 47.1 mm to (115.7, 103.5), turned to 90 degrees
- moved C44 44.4 mm to (113.2, 103.5), turned to 90 degrees
- moved R44 42.7 mm to (101.0, 117.3), turned to 180 degrees
- moved R45 41.8 mm to (97.4, 117.3), turned to 180 degrees
- moved R46 41.4 mm to (93.8, 117.3), turned to 0 degrees
- moved C46 40.6 mm to (105.2, 114.3), turned to 90 degrees
- moved R49 40.5 mm to (89.3, 116.3)
- moved R47 40.3 mm to (101.9, 115.3), turned to 0 degrees
- moved R48 38.0 mm to (89.3, 114.5), turned to 180 degrees
- moved C47 37.6 mm to (101.9, 113.3), turned to 0 degrees
- moved C39 36.6 mm to (84.4, 110.3), turned to 90 degrees
- moved U3 35.4 mm to (95.6, 112.9), turned to 0 degrees
- moved C40 34.3 mm to (87.7, 110.3), turned to 90 degrees
- moved C6 33.1 mm to (94.7, 86.9)
- moved J1 32.8 mm to (103.7, 86.3)
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Connections:
- U2 pad 4: +12VF -> Net-(U2-SHDN)
Routing:
- net +3V3_SYS: track 157.5 -> 81.4 mm, vias 17 -> 16
- net +3V3_CELL: track 100.0 -> 43.8 mm, vias 33 -> 14
- net CELL_PWR_EN: track 34.9 -> 66.8 mm
- net /~{MCLR}: track 49.8 -> 19.9 mm
- net /Power Protection/RAW_BATT: track 0.00 -> 28.0 mm
- net Net-(U1-RB7/ICSPDAT): track 47.8 -> 22.5 mm
- net Net-(U1-RB6/ICSPCLK): track 49.7 -> 26.4 mm
- net GND: track 57.6 -> 76.6 mm, vias 678 -> 695
- net Net-(U4-VCC): track 17.5 -> 0.00 mm
- net /Cellular/SIM_DET: track 60.3 -> 73.2 mm
- net CELL_PERST: track 72.8 -> 77.4 mm
- net +12VF: track 0.00 -> 4.08 mm, vias 26 -> 18
- net CELL_RI: track 83.0 -> 86.6 mm
- net Net-(D2-K): track 0.00 -> 3.40 mm
- net Net-(U2-SHDN): track 0.00 -> 2.96 mm
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- added copper zone on In2.Cu, net +3V3_CELL
- added copper zone on In2.Cu, net +3V3_SYS
- added copper zone on B.Cu, net GND
- added copper zone on In2.Cu, net GND
- removed copper zone on F.Cu, net +12VF
- removed copper zone on F.Cu, net /Power Protection/RAW_BATT
- removed copper zone on In2.Cu, net /Power Protection/RAW_BATT
- removed copper zone on F.Cu, net Net-(D1-K)
- removed copper zone on F.Cu, net Net-(D2-K)
- removed copper zone on F.Cu, net Net-(U4-VCC)
Other:
- board text added: "GNSS_RF_IN: 50R CPWG, W 0.34 / GAP 0.45, REF L2 (In1.Cu). CONTROLLED IMPEDANCE - STACKUP JLC04161H-7628"
