File: ki_cad_project/farseer/farseer.kicad_sch (KiCad schematic)
At the start: 20 parts, among them J1 Conn_PIC_ICSP_ICD, U1 PIC18F57Q84

Commit message: finished rev1
Parts:
- J1: footprint Connector_PinHeader_2.54mm:PinHeader_1x06_P2.54mm_Horizontal -> Connector_PinHeader_2.54mm:PinHeader_1x06_P2.54mm_Vertical
Changed lines of the file:
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@@
 			)
 		)
-		(property "Footprint" "Connector_PinHeader_2.54mm:PinHeader_1x06_P2.54mm_Horizontal"
+		(property "Footprint" "Connector_PinHeader_2.54mm:PinHeader_1x06_P2.54mm_Vertical"
 			(at 167.64 80.01 0)
 			(hide yes)
